File: KiCAD/PCB/YM60JIS_PCB.kicad_pcb (KiCad board)
At the start: 2 copper layers, 285.1 x 94.6 mm, 173 parts, among them J1 TYPE-C-31-M-12, SW1 SW_Push, SW10 SW_Push, SW11 SW_Push, SW12 SW_Push, SW13 SW_Push, SW14 SW_Push, SW15 SW_Push, SW16 SW_Push, SW17 SW_Push, SW18 SW_Push, SW19 SW_Push, SW2 SW_Push, SW20 SW_Push, SW21 SW_Push, SW22 SW_Push, SW23 SW_Push, SW24 SW_Push, SW25 SW_Push, SW26 SW_Push, SW27 SW_Push, SW28 SW_Push, SW29 Space, SW3 SW_Push, SW30 SW_Push, SW31 SW_Push, SW32 SW_Push, SW33 SW_Push, SW34 SW_Push, SW35 SW_Push, SW36 SW_Push, SW37 SW_Push, SW38 SW_Push, SW39 SW_Push, SW4 SW_Push, SW40 SW_Push, SW41 SW_Push, SW42 SW_Push, SW43 SW_Push, SW44 SW_Push, SW45 SW_Push, SW46 SW_Push, SW47 SW_Push, SW48 SW_Push, SW49 SW_Push, SW5 SW_Push, SW50 SW_Push, SW51 SW_Push, SW52 SW_Push, SW53 SW_Push, SW54 SW_Push, SW55 SW_Push, SW56 SW_Push, SW57 SW_Push, SW58 SW_Push, SW59 SW_Push, SW6 SW_Push, SW60 SW_Push, SW61 SW_Push, SW62 SW_Push, SW63 Yen, SW64 Backspace, SW65 ISOEnter, SW66 SW_Push, SW67 SW_Push, SW7 SW_Push, SW8 SW_Push, SW9 SW_Push, U1 XC6206P332MR, U2 SMF05CT1G, U3 RP2040, U4 W25Q16JVUXIQ, Y1 X322512MSB4SI

Commit message: reroute
Parts:
- removed REF**: STAB_MX_ISO, PCM_marbastlib-mx:STAB_MX_ISO
- removed REF**: STAB_MX_2.75u, PCM_marbastlib-mx:STAB_MX_2.75u
- removed REF**: STAB_MX_2u, PCM_marbastlib-mx:STAB_MX_2u
- removed REF**: STAB_MX_3u, PCM_marbastlib-mx:STAB_MX_3u
- added D68: D, Diode_SMD:D_SOD-123, B.Cu at (345.3, 138.1)
- added D69: D, Diode_SMD:D_SOD-123, B.Cu at (369.1, 138.1)
- added ST14: SW_stab, PCM_marbastlib-mx:STAB_MX_2u, F.Cu at (361.9, 57.1)
- added ST42: SW_stab, PCM_marbastlib-mx:STAB_MX_2u, F.Cu at (359.6, 95.2)
- added ST44: SW_stab, PCM_marbastlib-mx:STAB_MX_2u, F.Cu at (116.7, 114.3)
- added ST56: SW_stab, PCM_marbastlib-mx:STAB_MX_2u, F.Cu at (354.8, 114.3)
- added ST62: SW_stab, PCM_marbastlib-mx:STAB_MX_2u, F.Cu at (202.4, 133.3)
- added ST62_1: SW_stab, PCM_marbastlib-mx:STAB_MX_2u, F.Cu at (195.3, 133.3)
- added ST64: SW_stab, PCM_marbastlib-mx:STAB_MX_2u, F.Cu at (250.0, 133.3)
- added ST64_1: SW_stab, PCM_marbastlib-mx:STAB_MX_2u, F.Cu at (252.4, 133.4)
- added SW14_1: SW_Push, PCM_marbastlib-mx:SW_MX_HS_CPG151101S11_1u, B.Cu at (352.4, 57.1)
- added SW42_1: SW_Push, PCM_marbastlib-mx:SW_MX_HS_CPG151101S11_1.25u, B.Cu at (350.0, 95.2)
- added SW44_1: SW_Push, PCM_marbastlib-mx:SW_MX_HS_CPG151101S11_1u, B.Cu at (104.8, 114.3)
- added SW56_1: SW_Push, PCM_marbastlib-mx:SW_MX_HS_CPG151101S11_1.75u, B.Cu at (345.3, 114.3)
- added SW58_1: SW_Push, PCM_marbastlib-mx:SW_MX_HS_CPG151101S11_1u, B.Cu at (104.8, 133.3)
- added SW59_1: SW_Push, PCM_marbastlib-mx:SW_MX_HS_CPG151101S11_1.25u, B.Cu at (126.2, 133.3)
- added SW62_1: SW_Push, PCM_marbastlib-mx:SW_MX_HS_CPG151101S11_1u, B.Cu at (195.3, 133.3)
- added SW64_1: SW_Push, PCM_marbastlib-mx:SW_MX_HS_CPG151101S11_1u, B.Cu at (252.4, 133.4)
- added SW68: SW_Push, PCM_marbastlib-mx:SW_MX_HS_CPG151101S11_1.25u, B.Cu at (345.3, 133.3)
- added SW69: SW_Push, PCM_marbastlib-mx:SW_MX_HS_CPG151101S11_1.25u, B.Cu at (369.1, 133.3)
- D1, D10, D11, D12, D13, D14, D15, D16, D17, D18, D19, D2, D20, D21, D22, D23, D24, D25, D26, D27, D28, D29, D3, D30, D31, D32, D33, D34, D35, D36, D37, D38, D39, D4, D40, D41, D42, D43, D44, D45, D46, D47, D48, D49, D5, D50, D51, D52, D53, D54, D55, D56, D57, D58, D59, D6, D60, D61, D62, D63, D64, D65, D66, D67, D7, D8, D9: value 1N4148W -> D
- SW10, SW15, SW20, SW47, SW52: footprint PCM_marbastlib-mx:SW_MX_HS_CPG151101S11_1.25u -> PCM_marbastlib-mx:SW_MX_HS_CPG151101S11_1u
- SW16: footprint PCM_marbastlib-mx:SW_MX_HS_CPG151101S11_1u -> PCM_marbastlib-mx:SW_MX_HS_CPG151101S11_1.5u
- SW2, SW5: footprint PCM_marbastlib-mx:SW_MX_HS_CPG151101S11_1.5u -> PCM_marbastlib-mx:SW_MX_HS_CPG151101S11_1u
- SW29: value Space -> SW_Push; footprint PCM_marbastlib-mx:SW_MX_HS_CPG151101S11_1u -> PCM_marbastlib-mx:SW_MX_HS_CPG151101S11_1.5u
- SW3: footprint PCM_marbastlib-mx:SW_MX_HS_CPG151101S11_1.75u -> PCM_marbastlib-mx:SW_MX_HS_CPG151101S11_1u
- SW30: footprint PCM_marbastlib-mx:SW_MX_HS_CPG151101S11_1u -> PCM_marbastlib-mx:SW_MX_HS_CPG151101S11_1.75u
- SW45, SW58, SW67: footprint PCM_marbastlib-mx:SW_MX_HS_CPG151101S11_1u -> PCM_marbastlib-mx:SW_MX_HS_CPG151101S11_1.25u
- SW63: value Yen -> SW_Push
- SW64: value Backspace -> SW_Push
- SW65: value ISOEnter -> SW_Push
- moved SW58 238.7 mm to (107.2, 133.3), turned to 0 degrees
- moved D59 229.5 mm to (118.0, 126.7), turned to -90 degrees
- moved D58 227.7 mm to (115.1, 126.7), turned to -90 degrees
- moved SW15 225.2 mm to (371.5, 57.1), turned to 0 degrees
- moved SW59 221.8 mm to (128.6, 133.3), turned to 0 degrees
- moved D15 216.5 mm to (363.7, 66.2)
- moved SW14 208.0 mm to (361.9, 57.1)
- moved SW60 203.6 mm to (147.6, 133.3)
- moved D60 203.6 mm to (147.6, 138.1)
- moved D14 202.2 mm to (357.1, 66.2), turned to 180 degrees
- moved SW61 186.7 mm to (166.7, 133.3)
- moved D61 186.5 mm to (166.9, 138.0)
- moved D13 180.3 mm to (333.4, 61.9)
- moved SW13 180.3 mm to (333.4, 57.1)
- moved D44 179.2 mm to (111.5, 122.8), turned to 180 degrees
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Connections:
- D10 pad 1: ROW4 -> ROW0
- D12 pad 1: ROW1 -> ROW0
- D13 pad 1: ROW2 -> ROW0
- D14 pad 1: ROW3 -> ROW0
- D15 pad 1: ROW4 -> ROW0
- D16 pad 1: ROW0 -> ROW1
- D18 pad 1: ROW2 -> ROW1
- D19 pad 1: ROW3 -> ROW1
- D2 pad 1: ROW1 -> ROW0
- D20 pad 1: ROW4 -> ROW1
- D21 pad 1: ROW0 -> ROW1
- D23 pad 1: ROW2 -> ROW1
- D24 pad 1: ROW3 -> ROW1
- D25 pad 1: ROW0 -> ROW1
- D27 pad 1: ROW2 -> ROW1
- D28 pad 1: ROW3 -> ROW1
- D29 pad 1: ROW4 -> ROW1
- D3 pad 1: ROW2 -> ROW0
- D30 pad 1: ROW0 -> ROW2
- D31 pad 1: ROW1 -> ROW2
- D33 pad 1: ROW3 -> ROW2
- D34 pad 1: ROW0 -> ROW2
- D35 pad 1: ROW1 -> ROW2
- D37 pad 1: ROW3 -> ROW2
- D38 pad 1: ROW0 -> ROW2
- D39 pad 1: ROW1 -> ROW2
- D4 pad 1: ROW3 -> ROW0
- D41 pad 1: ROW3 -> ROW2
- D42 pad 1: ROW4 -> ROW2
- D43 pad 1: ROW0 -> ROW2
- D44 pad 1: ROW1 -> ROW3
- D45 pad 1: ROW2 -> ROW3
- D47 pad 1: ROW4 -> ROW3
- D48 pad 1: ROW0 -> ROW3
- D49 pad 1: ROW1 -> ROW3
- D5 pad 1: ROW4 -> ROW0
- D50 pad 1: ROW2 -> ROW3
- D52 pad 1: ROW4 -> ROW3
- D53 pad 1: ROW0 -> ROW3
- D54 pad 1: ROW1 -> ROW3
- D55 pad 1: ROW2 -> ROW3
- D57 pad 1: ROW4 -> ROW3
- D58 pad 1: ROW0 -> ROW4
- D59 pad 1: ROW1 -> ROW4
- D60 pad 1: ROW2 -> ROW4
- D61 pad 1: ROW3 -> ROW4
- D63 pad 1: ROW0 -> ROW4
- D64 pad 1: ROW1 -> ROW4
- D65 pad 1: ROW2 -> ROW4
- D66 pad 1: ROW3 -> ROW4
- D7 pad 1: ROW1 -> ROW0
- D8 pad 1: ROW2 -> ROW0
- D9 pad 1: ROW3 -> ROW0
- SW10 pad 1: COL1 -> COL9
- SW11 pad 1: COL2 -> COL10
- SW12 pad 1: COL2 -> COL11
- SW13 pad 1: COL2 -> COL12
- SW14 pad 1: COL2 -> COL13
- SW15 pad 1: COL2 -> COL14
- SW16 pad 1: COL3 -> COL0
- SW17 pad 1: COL3 -> COL1
- SW18 pad 1: COL3 -> COL2
- SW2 pad 1: COL0 -> COL1
- SW20 pad 1: COL3 -> COL4
- SW21 pad 1: COL4 -> COL5
- SW22 pad 1: COL4 -> COL6
- SW23 pad 1: COL4 -> COL7
- SW24 pad 1: COL4 -> COL8
- SW25 pad 1: COL5 -> COL9
- SW26 pad 1: COL5 -> COL10
- SW27 pad 1: COL5 -> COL11
- SW28 pad 1: COL5 -> COL12
- SW29 pad 1: COL5 -> Net-(D29-A)
- SW29 pad 2: Net-(D29-A) -> COL14
- SW3 pad 1: COL0 -> COL2
- SW30 pad 1: COL6 -> COL0
- SW31 pad 1: COL6 -> COL1
- SW32 pad 1: COL6 -> COL2
- SW33 pad 1: COL6 -> COL3
- SW34 pad 1: COL7 -> COL4
- SW35 pad 1: COL7 -> COL5
- SW36 pad 1: COL7 -> COL6
- SW39 pad 1: COL8 -> COL9
- SW4 pad 1: COL0 -> COL3
- SW40 pad 1: COL8 -> COL10
- SW41 pad 1: COL8 -> COL11
- SW42 pad 1: COL8 -> Net-(D42-A)
- SW42 pad 2: Net-(D42-A) -> COL13
- SW43 pad 1: COL9 -> COL14
- SW44 pad 1: COL9 -> Net-(D44-A)
- SW44 pad 2: Net-(D44-A) -> COL0
- SW45 pad 1: COL9 -> COL1
- SW46 pad 1: COL9 -> COL2
- SW47 pad 1: COL9 -> COL3
- SW48 pad 1: COL10 -> COL4
- SW49 pad 1: COL10 -> COL5
- SW5 pad 1: COL0 -> COL4
- SW50 pad 1: COL10 -> COL6
- SW51 pad 1: COL10 -> COL7
- SW52 pad 1: COL10 -> COL8
- SW53 pad 1: COL11 -> COL9
- SW54 pad 1: COL11 -> COL10
- SW56 pad 1: COL11 -> Net-(D56-A)
- SW56 pad 2: Net-(D56-A) -> COL13
- SW57 pad 1: COL11 -> COL14
- SW58 pad 1: COL12 -> Net-(D58-A)
- SW58 pad 2: Net-(D58-A) -> COL0
- SW59 pad 1: COL12 -> COL1
- SW6 pad 1: COL1 -> COL5
- SW60 pad 1: COL12 -> COL2
- SW61 pad 1: COL12 -> COL3
- SW62 pad 1: COL12 -> Net-(D62-A)
- SW62 pad 2: Net-(D62-A) -> COL5
- SW63 pad 1: COL13 -> COL6
- SW64 pad 1: COL13 -> COL7
- SW65 pad 1: COL13 -> COL9
- SW66 pad 1: COL13 -> COL10
- SW67 pad 1: COL13 -> COL11
- SW7 pad 1: COL1 -> COL6
- SW8 pad 1: COL1 -> COL7
- SW9 pad 1: COL1 -> COL8
- U3 pad 18: COL0 -> COL14
- U3 pad 37: unconnected-(U3-GPIO25-Pad37) -> COL0
Routing:
- net COL14: track 0.00 -> 368.2 mm, vias 0 -> 3
- net COL7: track 195.2 -> 238.1 mm
- net COL12: track 311.6 -> 275.9 mm
- net COL0: track 103.3 -> 134.6 mm, vias 2 -> 0
- net COL6: track 176.2 -> 203.1 mm
- net ROW3: track 368.4 -> 394.9 mm, vias 15 -> 16
- net COL5: track 178.2 -> 202.4 mm
- net ROW0: track 378.4 -> 397.5 mm
- net ROW2: track 376.9 -> 358.9 mm, vias 15 -> 14
- net COL8: track 238.1 -> 220.4 mm
- net Net-(D42-A): track 11.6 -> 27.7 mm
- net Net-(D56-A): track 11.6 -> 26.7 mm
- net Net-(D43-A): track 11.6 -> 26.0 mm
- net Net-(D64-A): track 11.6 -> 24.0 mm
- net Net-(D69-A): track 0.00 -> 11.6 mm
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
Commit message: reroute?
Parts:
- moved D17 10.3 mm to (143.6, 81.0)
- moved D64 4.98 mm to (264.4, 133.9)
- turned D18 to 0 degrees
- turned D27 to 180 degrees
Routing:
- net Net-(D64-A): track 24.0 -> 14.1 mm
- net ROW4: track 390.6 -> 395.3 mm

Commit message: address warnings
Parts:
- turned D16 to 0 degrees
- turned D27 to 0 degrees
Routing:
- net COL13: track 358.7 -> 346.5 mm
- net ROW4: track 395.3 -> 398.9 mm
- net Net-(D47-A): track 13.1 -> 11.6 mm
- net GND: vias 52 -> 51
