File: KiCAD/PCB/YM60JIS_PCB.kicad_pcb (KiCad board)
At the start: 2 copper layers, 285.1 x 94.6 mm, 189 parts, among them J1 TYPE-C-31-M-12, SW1 SW_Push, SW10 SW_Push, SW11 SW_Push, SW12 SW_Push, SW13 SW_Push, SW14 SW_Push, SW14_1 SW_Push, SW15 SW_Push, SW16 SW_Push, SW17 SW_Push, SW18 SW_Push, SW19 SW_Push, SW2 SW_Push, SW20 SW_Push, SW21 SW_Push, SW22 SW_Push, SW23 SW_Push, SW24 SW_Push, SW25 SW_Push, SW26 SW_Push, SW27 SW_Push, SW28 SW_Push, SW29 SW_Push, SW3 SW_Push, SW30 SW_Push, SW31 SW_Push, SW32 SW_Push, SW33 SW_Push, SW34 SW_Push, SW35 SW_Push, SW36 SW_Push, SW37 SW_Push, SW38 SW_Push, SW39 SW_Push, SW4 SW_Push, SW40 SW_Push, SW41 SW_Push, SW42 SW_Push, SW42_1 SW_Push, SW43 SW_Push, SW44 SW_Push, SW44_1 SW_Push, SW45 SW_Push, SW46 SW_Push, SW47 SW_Push, SW48 SW_Push, SW49 SW_Push, SW5 SW_Push, SW50 SW_Push, SW51 SW_Push, SW52 SW_Push, SW53 SW_Push, SW54 SW_Push, SW55 SW_Push, SW56 SW_Push, SW56_1 SW_Push, SW57 SW_Push, SW58 SW_Push, SW58_1 SW_Push, SW59 SW_Push, SW59_1 SW_Push, SW6 SW_Push, SW60 SW_Push, SW61 SW_Push, SW62 SW_Push, SW62_1 SW_Push, SW63 SW_Push, SW64 SW_Push, SW64_1 SW_Push, SW65 SW_Push, SW66 SW_Push, SW67 SW_Push, SW68 SW_Push, SW69 SW_Push, SW7 SW_Push, SW8 SW_Push, SW9 SW_Push, U1 XC6206P332MR, U2 SMF05CT1G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

Commit message: finish
Routing:
- net ROW1: track 336.5 -> 337.9 mm
- net GND: vias 51 -> 55
