File: KiCAD/PCB/YM60JIS_PCB.kicad_pcb (KiCad board)
At the start: 2 copper layers, 285.1 x 94.6 mm, 189 parts, among them J1 TYPE-C-31-M-12, SW1 SW_Push, SW10 SW_Push, SW11 SW_Push, SW12 SW_Push, SW13 SW_Push, SW14 SW_Push, SW14_1 SW_Push, SW15 SW_Push, SW16 SW_Push, SW17 SW_Push, SW18 SW_Push, SW19 SW_Push, SW2 SW_Push, SW20 SW_Push, SW21 SW_Push, SW22 SW_Push, SW23 SW_Push, SW24 SW_Push, SW25 SW_Push, SW26 SW_Push, SW27 SW_Push, SW28 SW_Push, SW29 SW_Push, SW3 SW_Push, SW30 SW_Push, SW31 SW_Push, SW32 SW_Push, SW33 SW_Push, SW34 SW_Push, SW35 SW_Push, SW36 SW_Push, SW37 SW_Push, SW38 SW_Push, SW39 SW_Push, SW4 SW_Push, SW40 SW_Push, SW41 SW_Push, SW42 SW_Push, SW42_1 SW_Push, SW43 SW_Push, SW44 SW_Push, SW44_1 SW_Push, SW45 SW_Push, SW46 SW_Push, SW47 SW_Push, SW48 SW_Push, SW49 SW_Push, SW5 SW_Push, SW50 SW_Push, SW51 SW_Push, SW52 SW_Push, SW53 SW_Push, SW54 SW_Push, SW55 SW_Push, SW56 SW_Push, SW56_1 SW_Push, SW57 SW_Push, SW58 SW_Push, SW58_1 SW_Push, SW59 SW_Push, SW59_1 SW_Push, SW6 SW_Push, SW60 SW_Push, SW61 SW_Push, SW62 SW_Push, SW62_1 SW_Push, SW63 SW_Push, SW64 SW_Push, SW64_1 SW_Push, SW65 SW_Push, SW66 SW_Push, SW67 SW_Push, SW68 SW_Push, SW69 SW_Push, SW7 SW_Push, SW8 SW_Push, SW9 SW_Push, U1 XC6206P332MR, U2 SMF05CT1G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

Commit message: exported production files
Parts:
- removed G***: LOGO, logo:ym60jis_logo_icononly
- removed G***: LOGO, logo:ym60jis_logo_ym60jis_only
Routing:
- net ROW2: track 359.4 -> 358.8 mm
Other:
- board text removed: "YM60JIS v1.1.1 @ymkn"

Commit message: snapshot: 2026-10-27 20:32:09+01:00
Parts:
- added ?: , , F.Cu at (223.4, 94.6)
- added SW44_2: SW_Push, PCM_marbastlib-mx:SW_MX_HS_CPG151101S11_1.25u, B.Cu at (107.2, 114.3)
- added SW45_1: SW_Push, PCM_marbastlib-mx:SW_MX_HS_CPG151101S11_1u, B.Cu at (128.6, 114.3)
- R6: value 1KΩ -> 1k
- R7: value 10kΩ -> 10k
- R8: value 1K -> 1k
- moved D36 6.63 mm to (233.2, 106.6), turned to 90 degrees
- moved D35 6.58 mm to (214.2, 106.6), turned to 90 degrees
- moved D45 1.82 mm to (115.9, 121.4)
- turned SW35 to -90 degrees
- turned SW36 to 90 degrees
Connections:
- SW35 pad 1: COL5 -> Net-(D35-A)
- SW35 pad 2: Net-(D35-A) -> COL5
Routing:
- net ROW3: track 394.9 -> 431.0 mm, vias 16 -> 15
- net COL6: track 203.1 -> 213.9 mm
- net ROW2: track 358.8 -> 368.4 mm
- net Net-(D35-A): track 11.6 -> 3.27 mm
- net Net-(D36-A): track 11.6 -> 6.35 mm
- net COL7: track 238.1 -> 242.6 mm
- net COL8: track 220.4 -> 224.3 mm
- net COL12: track 275.9 -> 279.8 mm
- net COL9: track 259.2 -> 263.1 mm
- net COL10: track 278.5 -> 282.2 mm
- net COL11: track 298.7 -> 302.3 mm
- net COL14: track 368.2 -> 371.4 mm
- net COL13: track 346.5 -> 349.4 mm
- net COL5: track 202.4 -> 200.2 mm
- net Net-(D44-A): track 13.4 -> 11.7 mm
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Other:
- board text added: "Unused case mount"
